Commit message: add joint limits

File: dexhand21s_description/urdf/dexhand21s.urdf.xacro (robot description, xacro)
@@ -51,5 +51,5 @@
     <child link="link_f_1_2" />
     <axis xyz="0 0 -1" />
-    <limit lower="-1.57" upper="1.57" effort="10.0" velocity="2.0" />
+    <limit lower="-1.3" upper="0.0" effort="10.0" velocity="2.0" />
   </joint>
   <link name="link_f_1_3">
@@ -86,5 +86,5 @@
     <child link="link_f_1_3" />
     <axis xyz="0 0 1" />
-    <limit lower="-1.57" upper="1.57" effort="10.0" velocity="2.0" />
+    <limit lower="0" upper="1.88" effort="10.0" velocity="2.0" />
   </joint>
   <link name="link_f_3_1">
@@ -156,5 +156,5 @@
     <child link="link_f_3_2" />
     <axis xyz="0 0 1" />
-    <limit lower="-1.57" upper="1.57" effort="10.0" velocity="2.0" />
+    <limit lower="0.0" upper="1.3" effort="10.0" velocity="2.0" />
   </joint>
   <link name="link_f_3_3">
@@ -191,5 +191,5 @@
     <child link="link_f_3_3" />
     <axis xyz="0 0 -1" />
-    <limit lower="-1.57" upper="1.57" effort="10.0" velocity="2.0" />
+    <limit lower="-1.88" upper="0.0" effort="10.0" velocity="2.0" />
   </joint>
   <link name="link_f_2_1">
@@ -261,5 +261,5 @@
     <child link="link_f_2_2" />
     <axis xyz="0 0 1" />
-    <limit lower="-1.57" upper="1.57" effort="10.0" velocity="2.0" />
+    <limit lower="0.0" upper="1.3" effort="10.0" velocity="2.0" />
   </joint>
   <link name="link_f_2_3">
@@ -296,5 +296,5 @@
     <child link="link_f_2_3" />
     <axis xyz="0 0 1" />
-    <limit lower="-1.57" upper="1.57" effort="10.0" velocity="2.0" />
+    <limit lower="0.0" upper="1.88" effort="10.0" velocity="2.0" />
   </joint>
 </robot>
